File: hardware/design/pi-eeprom-programmer.kicad_pcb (KiCad board)
At the start: 2 copper layers, 70 x 56 mm, 4 parts, among them J1 Raspberry Pi GPIO Connector, J2 Conn_01x03, U1 ZIF Socket, U2 24C01-24C1024

Commit message: Updated Version to 1.0.0 and generated new gerbers and zip
Other:
- board text added: "Ver. 1.0.0"
- board text removed: "Ver. 0.9.2"
Changed lines of the file:
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@@
   (title_block
     (title "Pi EEPROM Programmer")
-    (date "2023-08-20")
-    (rev "0.9.2")
+    (date "2023-12-04")
+    (rev "1.0.0")
   )
   (layers
@@
     (effects (font (size 1 1) (thickness 0.15)))
   )
-  (gr_text "Ver. 0.9.2" (at 166.878 83.142929 270) (layer "F.SilkS")
+  (gr_text "Ver. 1.0.0" (at 166.878 83.142929 270) (layer "F.SilkS")
     (effects (font (size 1 1) (thickness 0.15)))
   )
