File: hardware/design/pi-eeprom-programmer.kicad_sch (KiCad schematic)
At the start: 4 parts, among them J1 Raspberry Pi GPIO Connector, J2 Conn_01x03, U1 ZIF Socket, U2 24C01-24C1024

Commit message: Updated Version to 1.0.0 and generated new gerbers and zip
Other:
- title: Pi EEProm Programmer -> Pi EEPROM Programmer
Changed lines of the file:
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@@
   (paper "A4")
   (title_block
-    (title "Pi EEProm Programmer")
-    (date "2023-08-20")
-    (rev "0.9.2")
+    (title "Pi EEPROM Programmer")
+    (date "2023-12-04")
+    (rev "1.0.0")
   )
   (no_connect (at 100.33 66.04))
